Commit message: gripper.urdf.xacro

File: yale_hand_sim/putarm_driver/description/urdf/ur3_robot_puthand.urdf.xacro (robot description, xacro)
@@ -8,5 +8,5 @@
   <!-- arm -->
   <xacro:ur3_robot prefix="" joint_limited="false"/>
-  <link name="world" />
+  <link name="world"/>
   <joint name="world_joint" type="fixed">
     <parent link="world" />
@@ -15,6 +15,7 @@
   </joint>
    <!-- common stuff -->
-<!--  <xacro:include filename="$(find puthand_driver)/description/urdf/common.gazebo.xacro" /> -->
- <xacro:include filename="$(find wezelROS)/description/urdf/chwytak2.urdf.xacro" />
+<!--  <xacro:include filename="$(find puthand_driver)/description/urdf/common.gazebo.xacro" />
+  -->
+ <xacro:include filename="$(find node_yale_hand)/description/urdf/gripper.urdf.xacro" />
  <xacro:hand parent="ee_link" name="left_hand" side="-1">
     <origin xyz="0 0 0"  rpy= "0 1.57 0" />
