Commit message: gripper works

File: node_yale_hand/description/urdf/gripper.urdf.xacro (robot description, xacro)
@@ -1,5 +1,11 @@
 <?xml version="1.0"?>
-<robot name="gripper">
-  <link name="base_link">
+<robot xmlns:xacro="http://ros.org/wiki/xacro">
+  <xacro:macro name="gripperYale" params="parent name *origin">
+    <joint name="${name}_base_joint" type="fixed" >
+      <xacro:insert_block name="origin" />
+      <parent link="${parent}" />
+      <child link="gripper_base_link" />
+    </joint>
+  <link name="gripper_base_link">
     <visual>
       <geometry>
@@ -141,5 +147,5 @@
   </joint>
   <joint name="rotator2" type="continuous">
-    <parent link="base_link"/>
+    <parent link="gripper_base_link"/>
     <child link="rotator_link2"/>
     <axis xyz="0 0 1"/>
@@ -176,3 +182,4 @@
     <limit lower="-1.57" upper="1" effort="30" velocity="5"/>
   </joint>
+  </xacro:macro>
 </robot>

File: yale_hand_sim/putarm_driver/description/urdf/ur3_robot_puthand.urdf.xacro (robot description, xacro)
@@ -19,6 +19,6 @@
  <xacro:include filename="$(find node_yale_hand)/description/urdf/gripper.urdf.xacro" />
 <!--Error: unknown makro xacro:hand -->
- <xacro:hand parent="ee_link" name="left_hand" side="-1">
-    <origin xyz="0 0 0"  rpy= "0 1.57 0" />
-  </xacro:hand>
+ <xacro:gripperYale parent="ee_link" name="left_hand">
+    <origin xyz="0.1 0 0"  rpy= "0 1.57 0" />
+  </xacro:gripperYale>
 </robot>

Commit message: fixed joints

File: node_yale_hand/description/urdf/gripper.urdf.xacro (robot description, xacro)
@@ -12,5 +12,5 @@
         <mesh filename="package://node_yale_hand/description/meshes/base.dae"/>
       </geometry>
-      <origin xyz="0 0 0" rpy="1.57 0 3.14"/>
+      <origin xyz="0 0 0.01001" rpy="1.57 0 3.14"/>
     </visual>
     <collision>
@@ -141,5 +141,5 @@
   </link>
   <joint name="rotator1" type="fixed">
-    <parent link="base_link"/>
+    <parent link="gripper_base_link"/>
     <child link="rotator_link1"/>
     <axis xyz="0 0 1"/>
@@ -154,5 +154,5 @@
   </joint>
   <joint name="rotator3" type="continuous">
-    <parent link="base_link"/>
+    <parent link="gripper_base_link"/>
     <child link="rotator_link3"/>
     <axis xyz="0 0 1"/>

Commit message: moved gripper

File: node_yale_hand/description/urdf/gripper.urdf.xacro (robot description, xacro)
@@ -12,5 +12,5 @@
         <mesh filename="package://node_yale_hand/description/meshes/base.dae"/>
       </geometry>
-      <origin xyz="0 0 0.01001" rpy="1.57 0 3.14"/>
+      <origin xyz="0.0027 -0.009 0.01001" rpy="1.57 0 3.14"/>
     </visual>
     <collision>

Commit message: simulation works

File: node_yale_hand/description/urdf/gripper.urdf.xacro (robot description, xacro)
@@ -142,5 +142,5 @@
     </inertial>
   </link>
-  <joint name="rotator1" type="fixed">
+  <joint name="rotator1" type="continuous">
     <parent link="gripper_base_link"/>
     <child link="rotator_link1"/>
@@ -184,4 +184,6 @@
     <limit lower="-1.57" upper="1" effort="30" velocity="5"/>
   </joint>
+  <xacro:yale_hand_transmission name="${name}" />
+  <xacro:yale_hand_gazebo name="${name}" />
   </xacro:macro>
 </robot>

File: yale_hand_sim/putarm_driver/description/urdf/yale_hand.gazebo.xacro (robot description, xacro)
@@ -1,24 +1,24 @@
 <?xml version="1.0"?>
 <robot xmlns:xacro="http://ros.org/wiki/xacro">
-  <xacro:macro name="ur_arm_gazebo" params="prefix">
-    <gazebo reference="$gripper_base_link">
+  <xacro:macro name="yale_hand_gazebo" params="name">
+<!--    <gazebo reference="$gripper_base_link">
+      <selfCollide>true</selfCollide>
+    </gazebo>-->
+    <gazebo reference="rotator_link1">
       <selfCollide>true</selfCollide>
     </gazebo>
-    <gazebo reference="$rotator_link1">
+    <gazebo reference="rotator_link2">
       <selfCollide>true</selfCollide>
     </gazebo>
-    <gazebo reference="$rotator_link2">
+    <gazebo reference="rotator_link3">
       <selfCollide>true</selfCollide>
     </gazebo>
-    <gazebo reference="$rotator_link3">
+    <gazebo reference="finger_link1">
       <selfCollide>true</selfCollide>
     </gazebo>
-    <gazebo reference="$finger_link1">
+    <gazebo reference="finger_link2">
       <selfCollide>true</selfCollide>
     </gazebo>
-    <gazebo reference="$finger_link2">
-      <selfCollide>true</selfCollide>
-    </gazebo>
-    <gazebo reference="$finger_link3">
+    <gazebo reference="finger_link3">
       <selfCollide>true</selfCollide>
     </gazebo>

File: yale_hand_sim/putarm_driver/description/urdf/yale_hand.transmission.xacro (robot description, xacro)
@@ -1,6 +1,6 @@
 <?xml version="1.0"?>
 <robot xmlns:xacro="http://ros.org/wiki/xacro">
-  <xacro:macro name="yale_hand_transmission" params="prefix">
-    <transmission name="${name}_base_trans">
+  <xacro:macro name="yale_hand_transmission" params="name">
+<!--    <transmission name="${name}_base_trans">
       <type>transmission_interface/SimpleTransmission</type>
       <joint name="${name}_base_joint">
@@ -11,61 +11,61 @@
         <hardwareInterface>PositionJointInterface</hardwareInterface>
       </actuator>
-    </transmission>
-    <transmission name="$rotator1_trans">
+    </transmission>-->
+    <transmission name="rotator1_trans">
       <type>transmission_interface/SimpleTransmission</type>
-      <joint name="$rotator1">
+      <joint name="rotator1">
         <hardwareInterface>hardware_interface/PositionJointInterface</hardwareInterface>
       </joint>
-      <actuator name="$rotator1_motor">
+      <actuator name="rotator1_motor">
         <mechanicalReduction>1</mechanicalReduction>
         <hardwareInterface>PositionJointInterface</hardwareInterface>
       </actuator>
     </transmission>
-    <transmission name="$rotator2_trans">
+    <transmission name="rotator2_trans">
       <type>transmission_interface/SimpleTransmission</type>
-      <joint name="$rotator2">
+      <joint name="rotator2">
         <hardwareInterface>hardware_interface/PositionJointInterface</hardwareInterface>
       </joint>
-      <actuator name="$rotator2_motor">
+      <actuator name="rotator2_motor">
         <mechanicalReduction>1</mechanicalReduction>
         <hardwareInterface>PositionJointInterface</hardwareInterface>
       </actuator>
     </transmission>
-    <transmission name="$rotator3_trans">
+    <transmission name="rotator3_trans">
       <type>transmission_interface/SimpleTransmission</type>
-      <joint name="$rotator3">
+      <joint name="rotator3">
         <hardwareInterface>hardware_interface/PositionJointInterface</hardwareInterface>
       </joint>
-      <actuator name="$rotator3_motor">
+      <actuator name="rotator3_motor">
         <mechanicalReduction>1</mechanicalReduction>
         <hardwareInterface>PositionJointInterface</hardwareInterface>
       </actuator>
     </transmission>
-    <transmission name="$finger1_trans">
+    <transmission name="finger1_trans">
       <type>transmission_interface/SimpleTransmission</type>
-      <joint name="$finger1">
+      <joint name="finger1">
         <hardwareInterface>hardware_interface/PositionJointInterface</hardwareInterface>
       </joint>
-      <actuator name="$finger1_motor">
+      <actuator name="finger1_motor">
         <mechanicalReduction>1</mechanicalReduction>
         <hardwareInterface>PositionJointInterface</hardwareInterface>
       </actuator>
     </transmission>
-    <transmission name="$finger2_trans">
+    <transmission name="finger2_trans">
       <type>transmission_interface/SimpleTransmission</type>
-      <joint name="$finger2">
+      <joint name="finger2">
         <hardwareInterface>hardware_interface/PositionJointInterface</hardwareInterface>
       </joint>
-      <actuator name="$finger2_motor">
+      <actuator name="finger2_motor">
         <mechanicalReduction>1</mechanicalReduction>
         <hardwareInterface>PositionJointInterface</hardwareInterface>
       </actuator>
     </transmission>
-    <transmission name="$finger3_trans">
+    <transmission name="finger3_trans">
       <type>transmission_interface/SimpleTransmission</type>
-      <joint name="$finger3">
+      <joint name="finger3">
         <hardwareInterface>hardware_interface/PositionJointInterface</hardwareInterface>
       </joint>
-      <actuator name="$finger3_motor">
+      <actuator name="finger3_motor">
         <mechanicalReduction>1</mechanicalReduction>
         <hardwareInterface>PositionJointInterface</hardwareInterface>
