Commit message: control

File: hand_description/urdf/gripper.urdf.xacro (robot description, xacro)
@@ -12,5 +12,5 @@
     <visual>
       <geometry>
-        <mesh filename="package://node_yale_hand/description/meshes/base.dae"/>
+        <mesh filename="package://hand_description/meshes/base.dae"/>
       </geometry>
       <origin xyz="0.0027 -0.009 0.01001" rpy="1.57 0 3.14"/>
@@ -18,5 +18,5 @@
     <collision>
       <geometry>
-        <mesh filename="package://node_yale_hand/description/meshes/base.dae"/>
+        <mesh filename="package://hand_description/meshes/base.dae"/>
       </geometry>
       <origin xyz="0 0 0" rpy="1.57 0 3.14"/>
@@ -31,5 +31,5 @@
     <visual>
       <geometry>
-        <mesh filename="package://node_yale_hand/description/meshes/finger_rotator.dae"/>
+        <mesh filename="package://hand_description/meshes/finger_rotator.dae"/>
       </geometry>
       <origin xyz="0 0 0" rpy="1.57 0 0"/>
@@ -37,5 +37,5 @@
     <collision>
       <geometry>
-        <mesh filename="package://node_yale_hand/description/meshes/finger_rotator.dae"/>
+        <mesh filename="package://hand_description/meshes/finger_rotator.dae"/>
       </geometry>
       <origin xyz="0 0 0" rpy="1.57 0 0"/>
@@ -50,5 +50,5 @@
     <visual>
       <geometry>
-        <mesh filename="package://node_yale_hand/description/meshes/finger_rotator.dae"/>
+        <mesh filename="package://hand_description/meshes/finger_rotator.dae"/>
       </geometry>
       <origin xyz="0 0 0" rpy="1.57 0 3.14"/>
@@ -56,5 +56,5 @@
     <collision>
       <geometry>
-        <mesh filename="package://node_yale_hand/description/meshes/finger_rotator.dae"/>
+        <mesh filename="package://hand_description/meshes/finger_rotator.dae"/>
       </geometry>
       <origin xyz="0 0 0" rpy="1.57 0 3.14"/>
@@ -69,5 +69,5 @@
     <visual>
       <geometry>
-        <mesh filename="package://node_yale_hand/description/meshes/finger_rotator.dae"/>
+        <mesh filename="package://hand_description/meshes/finger_rotator.dae"/>
       </geometry>
       <origin xyz="0 0 0" rpy="1.57 0 3.14"/>
@@ -75,5 +75,5 @@
     <collision>
       <geometry>
-        <mesh filename="package://node_yale_hand/description/meshes/finger_rotator.dae"/>
+        <mesh filename="package://hand_description/meshes/finger_rotator.dae"/>
       </geometry>
       <origin xyz="0 0 0" rpy="1.57 0 3.14"/>
@@ -88,5 +88,5 @@
     <visual>
       <geometry>
-        <mesh filename="package://node_yale_hand/description/meshes/finger.dae"/>
+        <mesh filename="package://hand_description/meshes/finger.dae"/>
       </geometry>
       <origin xyz="0 0 0" rpy="1.57 0 0"/>
@@ -94,5 +94,5 @@
     <collision>
       <geometry>
-        <mesh filename="package://node_yale_hand/description/meshes/finger.dae"/>
+        <mesh filename="package://hand_description/meshes/finger.dae"/>
       </geometry>
       <origin xyz="0 0 0" rpy="1.57 0 0"/>
@@ -107,5 +107,5 @@
     <visual>
       <geometry>
-        <mesh filename="package://node_yale_hand/description/meshes/finger.dae"/>
+        <mesh filename="package://hand_description/meshes/finger.dae"/>
       </geometry>
       <origin xyz="0 0 0" rpy="1.57 0 3.14"/>
@@ -113,5 +113,5 @@
     <collision>
       <geometry>
-        <mesh filename="package://node_yale_hand/description/meshes/finger.dae"/>
+        <mesh filename="package://hand_description/meshes/finger.dae"/>
       </geometry>
       <origin xyz="0 0 0" rpy="1.57 0 3.14"/>
@@ -126,5 +126,5 @@
     <visual>
       <geometry>
-        <mesh filename="package://node_yale_hand/description/meshes/finger.dae"/>
+        <mesh filename="package://hand_description/meshes/finger.dae"/>
       </geometry>
       <origin xyz="0 0 0" rpy="1.57 0 3.14"/>
@@ -132,5 +132,5 @@
     <collision>
       <geometry>
-        <mesh filename="package://node_yale_hand/description/meshes/finger.dae"/>
+        <mesh filename="package://hand_description/meshes/finger.dae"/>
       </geometry>
       <origin xyz="0 0 0" rpy="1.57 0 3.14"/>

File: putarm_description/urdf/gripper.urdf.xacro (robot description, xacro)
@@ -12,5 +12,5 @@
     <visual>
       <geometry>
-        <mesh filename="package://node_yale_hand/description/meshes/base.dae"/>
+        <mesh filename="package://putarm_description/meshes/base.dae"/>
       </geometry>
       <origin xyz="0.0027 -0.009 0.01001" rpy="1.57 0 3.14"/>
@@ -18,5 +18,5 @@
     <collision>
       <geometry>
-        <mesh filename="package://node_yale_hand/description/meshes/base.dae"/>
+        <mesh filename="package://putarm_description/meshes/base.dae"/>
       </geometry>
       <origin xyz="0 0 0" rpy="1.57 0 3.14"/>
@@ -31,5 +31,5 @@
     <visual>
       <geometry>
-        <mesh filename="package://node_yale_hand/description/meshes/finger_rotator.dae"/>
+        <mesh filename="package://putarm_description/meshes/finger_rotator.dae"/>
       </geometry>
       <origin xyz="0 0 0" rpy="1.57 0 0"/>
@@ -37,5 +37,5 @@
     <collision>
       <geometry>
-        <mesh filename="package://node_yale_hand/description/meshes/finger_rotator.dae"/>
+        <mesh filename="package://putarm_description/meshes/finger_rotator.dae"/>
       </geometry>
       <origin xyz="0 0 0" rpy="1.57 0 0"/>
@@ -50,5 +50,5 @@
     <visual>
       <geometry>
-        <mesh filename="package://node_yale_hand/description/meshes/finger_rotator.dae"/>
+        <mesh filename="package://putarm_description/meshes/finger_rotator.dae"/>
       </geometry>
       <origin xyz="0 0 0" rpy="1.57 0 3.14"/>
@@ -56,5 +56,5 @@
     <collision>
       <geometry>
-        <mesh filename="package://node_yale_hand/description/meshes/finger_rotator.dae"/>
+        <mesh filename="package://putarm_description/meshes/finger_rotator.dae"/>
       </geometry>
       <origin xyz="0 0 0" rpy="1.57 0 3.14"/>
@@ -69,5 +69,5 @@
     <visual>
       <geometry>
-        <mesh filename="package://node_yale_hand/description/meshes/finger_rotator.dae"/>
+        <mesh filename="package://putarm_description/meshes/finger_rotator.dae"/>
       </geometry>
       <origin xyz="0 0 0" rpy="1.57 0 3.14"/>
@@ -75,5 +75,5 @@
     <collision>
       <geometry>
-        <mesh filename="package://node_yale_hand/description/meshes/finger_rotator.dae"/>
+        <mesh filename="package://putarm_description/meshes/finger_rotator.dae"/>
       </geometry>
       <origin xyz="0 0 0" rpy="1.57 0 3.14"/>
@@ -88,5 +88,5 @@
     <visual>
       <geometry>
-        <mesh filename="package://node_yale_hand/description/meshes/finger.dae"/>
+        <mesh filename="package://putarm_description/meshes/finger.dae"/>
       </geometry>
       <origin xyz="0 0 0" rpy="1.57 0 0"/>
@@ -94,5 +94,5 @@
     <collision>
       <geometry>
-        <mesh filename="package://node_yale_hand/description/meshes/finger.dae"/>
+        <mesh filename="package://putarm_description/meshes/finger.dae"/>
       </geometry>
       <origin xyz="0 0 0" rpy="1.57 0 0"/>
@@ -107,5 +107,5 @@
     <visual>
       <geometry>
-        <mesh filename="package://node_yale_hand/description/meshes/finger.dae"/>
+        <mesh filename="package://putarm_description/meshes/finger.dae"/>
       </geometry>
       <origin xyz="0 0 0" rpy="1.57 0 3.14"/>
@@ -113,5 +113,5 @@
     <collision>
       <geometry>
-        <mesh filename="package://node_yale_hand/description/meshes/finger.dae"/>
+        <mesh filename="package://putarm_description/meshes/finger.dae"/>
       </geometry>
       <origin xyz="0 0 0" rpy="1.57 0 3.14"/>
@@ -126,5 +126,5 @@
     <visual>
       <geometry>
-        <mesh filename="package://node_yale_hand/description/meshes/finger.dae"/>
+        <mesh filename="package://putarm_description/meshes/finger.dae"/>
       </geometry>
       <origin xyz="0 0 0" rpy="1.57 0 3.14"/>
@@ -132,5 +132,5 @@
     <collision>
       <geometry>
-        <mesh filename="package://node_yale_hand/description/meshes/finger.dae"/>
+        <mesh filename="package://putarm_description/meshes/finger.dae"/>
       </geometry>
       <origin xyz="0 0 0" rpy="1.57 0 3.14"/>
